Commit message: ROS Cartogarpher Setup

File: Software/ROS/Wheel_Robot/src/wheel_robot/urdf/wheel_robot.urdf (robot description, URDF)
Before this commit: robot fishbot, 7 links, 6 joints
Links:
- removed link base_footprint
- removed link caster_link
- link base_link: mass 0.2 -> 0.458809382377931; geometry collision mesh filename=package://wheel_robot/meshes/base_link.STL; visual mesh filename=package://wheel_robot/meshes/base_link.STL
- link imu_link: mass 0.1 -> 0.00215686283305885; geometry collision mesh filename=package://wheel_robot/meshes/imu_link.STL; visual mesh filename=package://wheel_robot/meshes/imu_link.STL
- link laser_link: mass 0.1 -> 0.0865823488601551; geometry collision mesh filename=package://wheel_robot/meshes/laser_link.STL; visual mesh filename=package://wheel_robot/meshes/laser_link.STL
- link left_wheel_link: mass 0.2 -> 0.016863123349881; geometry collision mesh filename=package://wheel_robot/meshes/left_wheel_link.STL; visual mesh filename=package://wheel_robot/meshes/left_wheel_link.STL
- link right_wheel_link: mass 0.2 -> 0.0168631232190387; geometry collision mesh filename=package://wheel_robot/meshes/right_wheel_link.STL; visual mesh filename=package://wheel_robot/meshes/right_wheel_link.STL
Joints:
- removed joint base_joint
- removed joint caster_joint
- joint imu_joint: axis (none) -> 0 0 0; origin xyz=0 0 0.02 -> xyz=-0.0100000000000001 0 0.094626149791491 rpy=0 0 0
- joint laser_joint: axis (none) -> 0 0 1; origin xyz=0 0 0.075 -> xyz=-0.000500000000000105 0 0.124626149791491 rpy=0 0 0
- joint left_wheel_joint: origin xyz=-0.02 0.10 -0.06 -> xyz=0 0.0655 0.0259589732744433 rpy=0 0 0
- joint right_wheel_joint: axis 0 1 0 -> 0 -1 0; origin xyz=-0.02 -0.10 -0.06 -> xyz=0 -0.0655 0.0259589732744432 rpy=0 0 0
